File: rfIMU.sch (EAGLE design)
At the start: 0 parts

Commit message: adds v2
Parts:
- added C1, C4: 10u, Brendan:CAP0603
- added C2, C3, C6: 0.1u, Brendan:CAP0603
- added C5: 1u, Brendan:CAP0603
- added IC1: TPS61201, texas:TPS61201
- added JP1: (no value), pinhead:PINHD-1X2
- added U1: (no value), esp8266modules:ESP12ESMD
- added U3: (no value), SparkFun-Sensors:MPU-9150QFN-24-NP
Connections:
- new net 3.3V: C1.2, C2.2, C3.2, C4.1, C4.2, C5.1, C5.2, C6.1, C6.2, IC1.FB, IC1.GND, IC1.PGND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
- new net N$2: C3.1, IC1.VAUX
- new net N$4: C1.1, C2.1, IC1.EN, IC1.UVLO, IC1.VIN
